Commit message: Environment and robot setup

File: hospital_ws/src/hospital_description/urdf/hospital_robot.urdf (robot description, URDF)
Before this commit: robot hospital_robot, 3 links, 2 joints
Links:
- added link front_caster, mass 0.1; collision sphere radius=0.05; visual sphere radius=0.05
- added link left_wheel, mass 0.5; collision cylinder length=0.04 radius=0.08; visual cylinder length=0.04 radius=0.08
- added link rear_caster, mass 0.1; collision sphere radius=0.05; visual sphere radius=0.05
- added link right_wheel, mass 0.5; collision cylinder length=0.04 radius=0.08; visual cylinder length=0.04 radius=0.08
- link base_link: mass None -> 5.0
- link camera_link: mass None -> 0.05; geometry collision box size=0.05 0.05 0.05; visual box size=0.05 0.05 0.05
- link lidar_link: mass None -> 0.2; geometry collision cylinder length=0.06 radius=0.05; visual cylinder length=0.06 radius=0.05
Joints:
- added joint front_caster_joint: type fixed, parent base_link, child front_caster, origin xyz=0.2 0 -0.05 rpy=0 0 0
- added joint left_wheel_joint: type continuous, parent base_link, child left_wheel, origin xyz=0.0 0.22 -0.02 rpy=0 0 0, axis 0 1 0
- added joint rear_caster_joint: type fixed, parent base_link, child rear_caster, origin xyz=-0.2 0 -0.05 rpy=0 0 0
- added joint right_wheel_joint: type continuous, parent base_link, child right_wheel, origin xyz=0.0 -0.22 -0.02 rpy=0 0 0, axis 0 1 0
- joint camera_joint: origin xyz=0.15 0 0.1 -> xyz=0.22 0 0.08 rpy=0 0 0
- joint lidar_joint: origin xyz=0 0 0.15 -> xyz=0 0 0.13 rpy=0 0 0
